Commit message: 1219

File: xacro/gazebo.xacro (robot description, xacro)
@@ -13,5 +13,5 @@
             <frequency>10</frequency>
             <plot>
-                <link>base</link>
+                <link>base_link</link>
                 <pose>0 0 0 0 0 0</pose>
                 <material>Gazebo/Yellow</material>
@@ -21,6 +21,6 @@
     <gazebo>
         <plugin filename="libgazebo_ros_force.so" name="gazebo_ros_force">
-            <bodyName>trunk</bodyName>
-            <topicName>/apply_force/trunk</topicName>
+            <bodyName>base_link</bodyName>
+            <topicName>/apply_force/base_link</topicName>
         </plugin>
     </gazebo>
@@ -48,5 +48,5 @@
         <turnGravityOff>false</turnGravityOff>
     </gazebo>
-    <gazebo reference="trunk">
+    <gazebo reference="base_link">
         <mu1>0.2</mu1>
         <mu2>0.2</mu2>

File: xacro/robot.xacro (robot description, xacro)
@@ -3,124 +3,349 @@
     <xacro:include filename="$(find livelybot_urdf)/xacro/const.xacro" />
     <xacro:include filename="$(find livelybot_urdf)/xacro/materials.xacro" />
-    <xacro:include filename="$(find livelybot_urdf)/xacro/leg.xacro" />
     <xacro:include filename="$(find livelybot_urdf)/xacro/stairs.xacro" />
     <xacro:include filename="$(find livelybot_urdf)/xacro/gazebo.xacro" />
+	<xacro:include filename="$(find livelybot_urdf)/xacro/transmission.xacro" />
     <!-- <xacro:stairs stairs="15" xpos="0" ypos="0" zpos="0" /> -->
-    <!-- Rollover Protection mode will add an additional stick on the top, use "true" or "false" to
-    switch it. -->
-    <xacro:property name="rolloverProtection" value="false" />
-    <!-- Debug mode will hung up the robot, use "true" or "false" to switch it. -->
-    <xacro:if value="$(arg DEBUG)">
-        <link name="world" />
-        <joint name="base_static_joint" type="fixed">
-            <origin rpy="0 0 0" xyz="0 0 0" />
-            <parent link="world" />
-            <child link="base" />
-        </joint>
-    </xacro:if>
-    <link name="base">
-        <visual>
-            <origin rpy="0 0 0" xyz="0 0 0" />
-            <geometry>
-                <box size="0.001 0.001 0.001" />
-            </geometry>
-        </visual>
-    </link>
-    <joint name="floating_base" type="fixed">
-        <origin rpy="0 0 0" xyz="0 0 0" />
-        <parent link="base" />
-        <child link="trunk" />
-    </joint>
-    <link name="trunk">
-        <visual>
-            <origin rpy="0 0 0" xyz="0 0 0" />
-            <geometry>
-                <mesh filename="package://livelybot_urdf/meshes/base_link.STL" scale="1 1 1"/>
-                <!-- <box size="${trunk_length*0.001} ${trunk_width*0.001} ${trunk_height*0.001}" /> -->
-            </geometry>
-            <material name="white" />
-        </visual>
-        <collision>
-            <origin rpy="0 0 0" xyz="0 0 0" />
-            <geometry>
-                <mesh filename="package://livelybot_urdf/meshes/base_link.STL" scale="1 1 1"/>
-                <!-- <box size="${trunk_length*0.001} ${trunk_width*0.001} ${trunk_height*0.001}" /> -->
-            </geometry>
-            <surface>
-                <contact>
-                    <ode>
-                        <min_depth>0.001</min_depth>
-                    </ode>
-                </contact>
-            </surface>
-        </collision>
-        <inertial>
-            <origin rpy="0 0 0" xyz="${trunk_com_x} ${trunk_com_y} ${trunk_com_z}" />
-            <mass value="${trunk_mass}" />
-            <inertia
-                ixx="${trunk_ixx*0.001*0.001}" ixy="${trunk_ixy*0.001*0.001}"
-                ixz="${trunk_ixz*0.001*0.001}"
-                iyy="${trunk_iyy*0.001*0.001}" iyz="${trunk_iyz*0.001*0.001}"
-                izz="${trunk_izz*0.001*0.001}" />
-        </inertial>
-    </link>
-    <xacro:if value="${(rolloverProtection == 'True')}">
-        <joint name="stick_joint" type="fixed">
-            <parent link="trunk" />
-            <child link="stick_link" />
-            <origin rpy="0 0 0" xyz="${0.18} 0 ${stick_length/2.0+0.08}" />
-        </joint>
-        <link name="stick_link">
-            <visual>
-                <geometry>
-                    <cylinder length="${stick_length}" radius="${stick_radius}" />
-                </geometry>
-                <origin rpy="0 0 0" xyz="0 0 0" />
-                <material name="white" />
-            </visual>
-            <collision>
-                <geometry>
-                    <cylinder length="${stick_length}" radius="${stick_radius}" />
-                </geometry>
-                <origin rpy="0 0 0" xyz="0 0 0" />
-            </collision>
-            <inertial>
-                <mass value="${stick_mass}" />
-                <inertia
-                    ixx="${stick_mass / 2.0 * (stick_radius*stick_radius)}" ixy="0.0" ixz="0.0"
-                    iyy="${stick_mass / 12.0 * (3*stick_radius*stick_radius + stick_length*stick_length)}"
-                    iyz="0.0"
-                    izz="${stick_mass / 12.0 * (3*stick_radius*stick_radius + stick_length*stick_length)}" />
-            </inertial>
-        </link>
-    </xacro:if>
-    <joint name="imu_joint" type="fixed">
-        <parent link="trunk" />
-        <child link="imu_link" />
-        <origin rpy="0 0 ${PI}" xyz="0 0 0" />
-    </joint>
-    <link name="imu_link">
-        <inertial>
-            <mass value="0.001" />
-            <origin rpy="0 0 0" xyz="0 0 0" />
-            <inertia ixx="0.0001" ixy="0" ixz="0" iyy="0.0001" iyz="0" izz="0.0001" />
-        </inertial>
-        <visual>
-            <origin rpy="0 0 0" xyz="0 0 0" />
-            <geometry>
-                <box size="0.001 0.001 0.001" />
-            </geometry>
-            <material name="red" />
-        </visual>
-        <collision>
-            <origin rpy="0 0 0" xyz="0 0 0" />
-            <geometry>
-                <box size=".001 .001 .001" />
-            </geometry>
-        </collision>
-    </link>
-    <xacro:leg name="L" mirror="1" mirror_dae="False">
-    </xacro:leg>
-    <xacro:leg name="R" mirror="-1" mirror_dae="True">
-    </xacro:leg>
+    <link name="base_link">
+		<inertial>
+			<origin xyz="0.042418 -5.836E-05 0.017336" rpy="0 0 0" />
+			<mass value="0.63088" />
+			<inertia ixx="0.0019802" ixy="3.6377E-08" ixz="3.091E-05" iyy="0.0011784" iyz="2.0119E-08" izz="0.0024461" />
+		</inertial>
+		<visual>
+			<origin xyz="0 0 0" rpy="0 0 0" />
+			<geometry>
+				<mesh filename="package://livelybot_urdf/meshes/base_link.STL" />
+			</geometry>
+			<material name="">
+				<color rgba="1 1 1 1" />
+			</material>
+		</visual>
+		<collision>
+			<origin xyz="0 0 0" rpy="0 0 0" />
+			<geometry>
+				<mesh filename="package://livelybot_urdf/meshes/base_link.STL" />
+			</geometry>
+		</collision>
+	</link>
+	<link name="imu_link">
+		<inertial>
+			<origin xyz="0.0137089490024808 -2.94548196346016E-05 -0.0923185931780866" rpy="0 0 0" />
+			<mass value="4.769" />
+			<inertia ixx="0.0808092488138549" ixy="8.98366603728616E-06" ixz="-0.00786465247064748" iyy="0.0675694550274403" iyz="1.41271229184058E-05" izz="0.0287128301147392" />
+		</inertial>
+		<visual>
+			<origin xyz="0 0 0" rpy="0 0 0" />
+			<geometry>
+        <box size="0.001 0.001 0.001" />
+			</geometry>
+			<material name="">
+				<color rgba="1 1 1 1" />
+			</material>
+		</visual>
+		<collision>
+			<origin xyz="0 0 0" rpy="0 0 0" />
+			<geometry>
+        <box size="0.001 0.001 0.001" />
+			</geometry>
+		</collision>
+	</link>
+	<joint name="base_imu_joint" type="fixed">
+		<origin xyz="0 0 0.00572" rpy="0 0 0" />
+		<parent link="base_link" />
+		<child link="imu_link" />
+		<axis xyz="0 0 0" />
+	</joint>
+	<link name="L_hip">
+		<inertial>
+			<origin xyz="0.0560469785532357 -6.40933923989895E-09 0.0465742815241479" rpy="0 0 0" />
+			<mass value="0.116884292970712" />
+			<inertia ixx="3.7540266331977E-05" ixy="-9.42771492040107E-12" ixz="-4.36077137816932E-06" iyy="4.69555171175074E-05" iyz="-2.72493557400722E-12" izz="4.32454239525254E-05" />
+		</inertial>
+		<visual>
+			<origin xyz="0 0 0" rpy="0 0 0" />
+			<geometry>
+				<mesh filename="package://livelybot_urdf/meshes/L_hip.STL" />
+			</geometry>
+			<material name="">
+				<color rgba="1 1 1 1" />
+			</material>
+		</visual>
+		<collision>
+			<origin xyz="0 0 0" rpy="0 0 0" />
+			<geometry>
+				<mesh filename="package://livelybot_urdf/meshes/L_hip.STL" />
+			</geometry>
+		</collision>
+	</link>
+	<joint name="L_hip_joint" type="revolute">
+		<origin xyz="0 0.075 0" rpy="3.1416 0 3.1416" />
+		<parent link="base_link" />
+		<child link="L_hip" />
+		<axis xyz="0 0 -1" />
+		<limit lower="-0.55" upper="0.55" effort="0" velocity="0" />
+	</joint>
+	<link name="L_hip2">
+		<inertial>
+			<origin xyz="0.0309072230654156 -0.000858756081910141 0.0332451481987078" rpy="0 0 0" />
+			<mass value="0.125448617656537" />
+			<inertia ixx="5.53521193479647E-05" ixy="-3.56340330502834E-06" ixz="-1.93226894229574E-05" iyy="7.99417228381797E-05" iyz="-1.84997816876284E-06" izz="6.64062940642034E-05" />
+		</inertial>
+		<visual>
+			<origin xyz="0 0 0" rpy="0 0 0" />
+			<geometry>
+				<mesh filename="package://livelybot_urdf/meshes/L_hip2.STL" />
+			</geometry>
+			<material name="">
+				<color rgba="1 1 1 1" />
+			</material>
+		</visual>
+		<collision>
+			<origin xyz="0 0 0" rpy="0 0 0" />
+			<geometry>
+				<mesh filename="package://livelybot_urdf/meshes/L_hip2.STL" />
+			</geometry>
+		</collision>
+	</link>
+	<joint name="L_hip2_joint" type="revolute">
+		<origin xyz="0.037 0 0.054" rpy="-1.5708 0 1.5708" />
+		<parent link="L_hip" />
+		<child link="L_hip2" />
+		<axis xyz="0 0 -1" />
+		<limit lower="-0.48" upper="0.18" effort="0" velocity="0" />
+	</joint>
+	<link name="L_thigh">
+		<inertial>
+			<origin xyz="0.0223260729573922 3.03576608295941E-18 0.0400536863070936" rpy="0 0 0" />
+			<mass value="0.137807983904981" />
+			<inertia ixx="4.68049989970575E-05" ixy="-4.55991575251683E-20" ixz="3.01249192067359E-05" iyy="0.000231171478895831" iyz="8.22464509411909E-21" izz="0.000224309841397752" />
+		</inertial>
+		<visual>
+			<origin xyz="0 0 0" rpy="0 0 0" />
+			<geometry>
+				<mesh filename="package://livelybot_urdf/meshes/L_thigh.STL" />
+			</geometry>
+			<material name="">
+				<color rgba="1 1 1 1" />
+			</material>
+		</visual>
+		<collision>
+			<origin xyz="0 0 0" rpy="0 0 0" />
+			<geometry>
+				<mesh filename="package://livelybot_urdf/meshes/L_thigh.STL" />
+			</geometry>
+		</collision>
+	</link>
+	<joint name="L_thigh_joint" type="revolute">
+		<origin xyz="0.0161 0 0.039" rpy="1.5708 0 -1.5708" />
+		<parent link="L_hip2" />
+		<child link="L_thigh" />
+		<axis xyz="0 0 -1" />
+		<limit lower="-1.0" upper="0.44" effort="0" velocity="0" />
+	</joint>
+	<link name="L_calf">
+		<inertial>
+			<origin xyz="0.0637217850662202 0.0045962102584563 0.0125678073048835" rpy="0 0 0" />
+			<mass value="0.106343448636289" />
+			<inertia ixx="2.00356805610283E-05" ixy="3.32248264945443E-07" ixz="-1.28437033439576E-07" iyy="0.000119450065875996" iyz="-6.40774201031294E-08" izz="0.000122526027150439" />
+		</inertial>
+		<visual>
+			<origin xyz="0 0 0" rpy="0 0 0" />
+			<geometry>
+				<mesh filename="package://livelybot_urdf/meshes/L_calf.STL" />
+			</geometry>
+			<material name="">
+				<color rgba="1 1 1 1" />
+			</material>
+		</visual>
+		<collision>
+			<origin xyz="0 0 0" rpy="0 0 0" />
+			<geometry>
+				<mesh filename="package://livelybot_urdf/meshes/L_calf.STL" />
+			</geometry>
+		</collision>
+	</link>
+	<joint name="L_calf_joint" type="revolute">
+		<origin xyz="0.15 0 0.0161" rpy="-3.1416 0 0" />
+		<parent link="L_thigh" />
+		<child link="L_calf" />
+		<axis xyz="0 0 1" />
+		<limit lower="0.0" upper="2.0" effort="0" velocity="0" />
+	</joint>
+	<link name="L_toe">
+		<inertial>
+			<origin xyz="0.000834584120334044 -0.0112941816613386 6.46892758804363E-09" rpy="0 0 0" />
+			<mass value="0.0187301054238791" />
+			<inertia ixx="1.17270430762399E-06" ixy="6.03537221578576E-07" ixz="1.89483242400211E-14" iyy="1.08896121231129E-05" iyz="3.6633857520274E-22" izz="1.12731889139232E-05" />
+		</inertial>
+		<visual>
+			<origin xyz="0 0 0" rpy="0 0 0" />
+			<geometry>
+				<mesh filename="package://livelybot_urdf/meshes/L_toe.STL" />
+			</geometry>
+			<material name="">
+				<color rgba="1 1 1 1" />
+			</material>
+		</visual>
+		<collision>
+			<origin xyz="0 0 0" rpy="0 0 0" />
+			<geometry>
+				<mesh filename="package://livelybot_urdf/meshes/L_toe.STL" />
+			</geometry>
+		</collision>
+	</link>
+	<joint name="L_toe_joint" type="revolute">
+		<origin xyz="0.16 0 0" rpy="-3.1416 0 -1.5708" />
+		<parent link="L_calf" />
+		<child link="L_toe" />
+		<axis xyz="0 0 1" />
+		<limit lower="-0.85" upper="1.0" effort="0" velocity="0" />
+	</joint>
+	<link name="R_hip">
+		<inertial>
+			<origin xyz="0.0560469785532357 -6.40933922602116E-09 0.0465742815241478" rpy="0 0 0" />
+			<mass value="0.116884292970712" />
+			<inertia ixx="3.7540266331977E-05" ixy="-9.42771492313437E-12" ixz="-4.36077137816932E-06" iyy="4.69555171175074E-05" iyz="-2.72493557242105E-12" izz="4.32454239525254E-05" />
+		</inertial>
+		<visual>
+			<origin xyz="0 0 0" rpy="0 0 0" />
+			<geometry>
+				<mesh filename="package://livelybot_urdf/meshes/R_hip.STL" />
+			</geometry>
+			<material name="">
+				<color rgba="1 1 1 1" />
+			</material>
+		</visual>
+		<collision>
+			<origin xyz="0 0 0" rpy="0 0 0" />
+			<geometry>
+				<mesh filename="package://livelybot_urdf/meshes/R_hip.STL" />
+			</geometry>
+		</collision>
+	</link>
+	<joint name="R_hip_joint" type="revolute">
+		<origin xyz="0 -0.075 0" rpy="3.1416 0 3.1416" />
+		<parent link="base_link" />
+		<child link="R_hip" />
+		<axis xyz="0 0 -1" />
+		<limit lower="-0.55" upper="0.55" effort="0" velocity="0" />
+	</joint>
+	<link name="R_hip2">
+		<inertial>
+			<origin xyz="0.0309072116551233 0.000858757175953094 0.0332451451614201" rpy="0 0 0" />
+			<mass value="0.125448645563517" />
+			<inertia ixx="5.53521261009191E-05" ixy="3.56340110481497E-06" ixz="-1.93227169282725E-05" iyy="7.99417985454008E-05" iyz="1.8499802142557E-06" izz="6.64063646851793E-05" />
+		</inertial>
+		<visual>
+			<origin xyz="0 0 0" rpy="0 0 0" />
+			<geometry>
+				<mesh filename="package://livelybot_urdf/meshes/R_hip2.STL" />
+			</geometry>
+			<material name="">
+				<color rgba="1 1 1 1" />
+			</material>
+		</visual>
+		<collision>
+			<origin xyz="0 0 0" rpy="0 0 0" />
+			<geometry>
+				<mesh filename="package://livelybot_urdf/meshes/R_hip2.STL" />
+			</geometry>
+		</collision>
+	</link>
+	<joint name="R_hip2_joint" type="revolute">
+		<origin xyz="0.037 0 0.054" rpy="1.5708 0 -1.5708" />
+		<parent link="R_hip" />
+		<child link="R_hip2" />
+		<axis xyz="0 0 -1" />
+		<limit lower="-0.18" upper="0.48" effort="0" velocity="0" />
+	</joint>
+	<link name="R_thigh">
+		<inertial>
+			<origin xyz="0.0223260729573922 4.33680868994202E-19 0.0400536863070936" rpy="0 0 0" />
+			<mass value="0.137807983904981" />
+			<inertia ixx="4.68049989970575E-05" ixy="1.39680883168296E-21" ixz="3.01249192067358E-05" iyy="0.00023117147889583" iyz="1.89032544259718E-21" izz="0.000224309841397752" />
+		</inertial>
+		<visual>
+			<origin xyz="0 0 0" rpy="0 0 0" />
+			<geometry>
+				<mesh filename="package://livelybot_urdf/meshes/R_thigh.STL" />
+			</geometry>
+			<material name="">
+				<color rgba="1 1 1 1" />
+			</material>
+		</visual>
+		<collision>
+			<origin xyz="0 0 0" rpy="0 0 0" />
+			<geometry>
+				<mesh filename="package://livelybot_urdf/meshes/R_thigh.STL" />
+			</geometry>
+		</collision>
+	</link>
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