Commit message: 1220

File: xacro/robot.xacro (robot description, xacro)
@@ -84,5 +84,5 @@
 		<child link="L_hip" />
 		<axis xyz="0 0 -1" />
-		<limit lower="-0.55" upper="0.55" effort="0" velocity="0" />
+		<limit lower="-0.55" upper="0.55" effort="20.0" velocity="20.0" />
 	</joint>
 	<link name="L_hip2">
@@ -113,5 +113,5 @@
 		<child link="L_hip2" />
 		<axis xyz="0 0 -1" />
-		<limit lower="-0.48" upper="0.18" effort="0" velocity="0" />
+		<limit lower="-0.48" upper="0.18" effort="20.0" velocity="20.0" />
 	</joint>
 	<link name="L_thigh">
@@ -142,5 +142,5 @@
 		<child link="L_thigh" />
 		<axis xyz="0 0 -1" />
-		<limit lower="-1.0" upper="0.44" effort="0" velocity="0" />
+		<limit lower="-1.0" upper="0.44" effort="20.0" velocity="20.0" />
 	</joint>
 	<link name="L_calf">
@@ -171,5 +171,5 @@
 		<child link="L_calf" />
 		<axis xyz="0 0 1" />
-		<limit lower="0.0" upper="2.0" effort="0" velocity="0" />
+		<limit lower="0.0" upper="2.0" effort="20.0" velocity="20.0" />
 	</joint>
 	<link name="L_toe">
@@ -200,5 +200,5 @@
 		<child link="L_toe" />
 		<axis xyz="0 0 1" />
-		<limit lower="-0.85" upper="1.0" effort="0" velocity="0" />
+		<limit lower="-0.85" upper="1.0" effort="20.0" velocity="20.0" />
 	</joint>
 	<link name="R_hip">
@@ -229,5 +229,5 @@
 		<child link="R_hip" />
 		<axis xyz="0 0 -1" />
-		<limit lower="-0.55" upper="0.55" effort="0" velocity="0" />
+		<limit lower="-0.55" upper="0.55" effort="20.0" velocity="20.0" />
 	</joint>
 	<link name="R_hip2">
@@ -258,5 +258,5 @@
 		<child link="R_hip2" />
 		<axis xyz="0 0 -1" />
-		<limit lower="-0.18" upper="0.48" effort="0" velocity="0" />
+		<limit lower="-0.18" upper="0.48" effort="20.0" velocity="20.0" />
 	</joint>
 	<link name="R_thigh">
@@ -287,5 +287,5 @@
 		<child link="R_thigh" />
 		<axis xyz="0 0 -1" />
-		<limit lower="-0.44" upper="1.0" effort="0" velocity="0" />
+		<limit lower="-0.44" upper="1.0" effort="20.0" velocity="20.0" />
 	</joint>
 	<link name="R_calf">
@@ -316,5 +316,5 @@
 		<child link="R_calf" />
 		<axis xyz="0 0 1" />
-		<limit lower="-2.0" upper="0" effort="0" velocity="0" />
+		<limit lower="-2.0" upper="0" effort="20.0" velocity="20.0" />
 	</joint>
 	<link name="R_toe">
@@ -345,5 +345,5 @@
 		<child link="R_toe" />
 		<axis xyz="0 0 1" />
-		<limit lower="-1.0" upper="0.85" effort="0" velocity="0" />
+		<limit lower="-1.0" upper="0.85" effort="20.0" velocity="20.0" />
 	</joint>
 	<xacro:leg_transmission name="R" />

Commit message: 0106

File: xacro/robot.xacro (robot description, xacro)
@@ -32,6 +32,6 @@
 		<inertial>
 			<origin xyz="0.0137089490024808 -2.94548196346016E-05 -0.0923185931780866" rpy="0 0 0" />
-			<mass value="4.769" />
-			<inertia ixx="0.0808092488138549" ixy="8.98366603728616E-06" ixz="-0.00786465247064748" iyy="0.0675694550274403" iyz="1.41271229184058E-05" izz="0.0287128301147392" />
+			<mass value="0.0" />
+			<inertia ixx="0.0" ixy="0.0" ixz="0.0" iyy="0.0" iyz="0.0" izz="0.0" />
 		</inertial>
 		<visual>
