Commit message: 0107

File: urdf/livelybot_urdf.urdf (robot description, URDF)
Before this commit: robot livelybot_urdf, 12 links, 11 joints
Links:
- link imu_link: mass 4.769 -> 0.0
Joints:
- joint L_calf_joint: limit lower=0.0 upper=2.0 effort=0 velocity=0 -> lower=0.0 upper=1.7 effort=20.0 velocity=20.0; origin xyz=0.15 0 0.0161 rpy=-3.1416 0 0 -> xyz=0.15 0 0.0161 rpy=-3.1416 0 -0.5
- joint L_hip2_joint: axis 0 0 -1 -> 0 0 1; limit lower=-0.48 upper=0.18 effort=0 velocity=0 -> lower=-0.18 upper=0.48 effort=20.0 velocity=20.0
- joint L_hip_joint: axis 0 0 -1 -> 0 0 1; limit lower=-0.55 upper=0.55 effort=0 velocity=0 -> lower=-0.55 upper=0.55 effort=20.0 velocity=20.0
- joint L_thigh_joint: axis 0 0 -1 -> 0 0 1; limit lower=-1.0 upper=0.44 effort=0 velocity=0 -> lower=-0.44 upper=1.0 effort=20.0 velocity=20.0; origin xyz=0.0161 0 0.039 rpy=1.5708 0 -1.5708 -> xyz=0.0161 0 0.039 rpy=1.5708 -0.25 -1.5708
- joint L_toe_joint: limit lower=-0.85 upper=1.0 effort=0 velocity=0 -> lower=-0.85 upper=1.0 effort=20.0 velocity=20.0; origin xyz=0.16 0 0 rpy=-3.1416 0 -1.5708 -> xyz=0.16 0 0 rpy=-3.1416 0 -1.8208
- joint R_calf_joint: limit lower=-2.0 upper=0 effort=0 velocity=0 -> lower=-1.7 upper=0 effort=20.0 velocity=20.0; origin xyz=0.15 0 0.0161 rpy=3.1416 0 0 -> xyz=0.15 0 0.0161 rpy=3.1416 0 0.5
- joint R_hip2_joint: axis 0 0 -1 -> 0 0 1; limit lower=-0.18 upper=0.48 effort=0 velocity=0 -> lower=-0.48 upper=0.18 effort=20.0 velocity=20.0
- joint R_hip_joint: axis 0 0 -1 -> 0 0 1; limit lower=-0.55 upper=0.55 effort=0 velocity=0 -> lower=-0.55 upper=0.55 effort=20.0 velocity=20.0
- joint R_thigh_joint: axis 0 0 -1 -> 0 0 1; limit lower=-0.44 upper=1.0 effort=0 velocity=0 -> lower=-1.0 upper=0.44 effort=20.0 velocity=20.0; origin xyz=0.0161 0 0.039 rpy=-1.5708 0 1.5708 -> xyz=0.0161 0 0.039 rpy=-1.5708 -0.25 1.5708
- joint R_toe_joint: limit lower=-1.0 upper=0.85 effort=0 velocity=0 -> lower=-1.0 upper=0.85 effort=20.0 velocity=20.0; origin xyz=0.16 0 0 rpy=3.1416 0 1.5708 -> xyz=0.16 0 0 rpy=3.1416 0 1.8208

File: xacro/robot.xacro (robot description, xacro)
@@ -83,5 +83,5 @@
 		<parent link="base_link" />
 		<child link="L_hip" />
-		<axis xyz="0 0 -1" />
+		<axis xyz="0 0 1" />
 		<limit lower="-0.55" upper="0.55" effort="20.0" velocity="20.0" />
 	</joint>
@@ -112,6 +112,6 @@
 		<parent link="L_hip" />
 		<child link="L_hip2" />
-		<axis xyz="0 0 -1" />
-		<limit lower="-0.48" upper="0.18" effort="20.0" velocity="20.0" />
+		<axis xyz="0 0 1" />
+		<limit lower="-0.18" upper="0.48" effort="20.0" velocity="20.0" />
 	</joint>
 	<link name="L_thigh">
@@ -138,9 +138,9 @@
 	</link>
 	<joint name="L_thigh_joint" type="revolute">
-		<origin xyz="0.0161 0 0.039" rpy="1.5708 0 -1.5708" />
+		<origin xyz="0.0161 0 0.039" rpy="1.5708 -0.25 -1.5708" />
 		<parent link="L_hip2" />
 		<child link="L_thigh" />
-		<axis xyz="0 0 -1" />
-		<limit lower="-1.0" upper="0.44" effort="20.0" velocity="20.0" />
+		<axis xyz="0 0 1" />
+		<limit lower="-0.44" upper="1.0" effort="20.0" velocity="20.0" />
 	</joint>
 	<link name="L_calf">
@@ -167,9 +167,9 @@
 	</link>
 	<joint name="L_calf_joint" type="revolute">
-		<origin xyz="0.15 0 0.0161" rpy="-3.1416 0 0" />
+		<origin xyz="0.15 0 0.0161" rpy="-3.1416 0 -0.5" />
 		<parent link="L_thigh" />
 		<child link="L_calf" />
 		<axis xyz="0 0 1" />
-		<limit lower="0.0" upper="2.0" effort="20.0" velocity="20.0" />
+		<limit lower="0.0" upper="1.7" effort="20.0" velocity="20.0" />
 	</joint>
 	<link name="L_toe">
@@ -196,5 +196,5 @@
 	</link>
 	<joint name="L_toe_joint" type="revolute">
-		<origin xyz="0.16 0 0" rpy="-3.1416 0 -1.5708" />
+		<origin xyz="0.16 0 0" rpy="-3.1416 0 -1.8208" />
 		<parent link="L_calf" />
 		<child link="L_toe" />
@@ -228,5 +228,5 @@
 		<parent link="base_link" />
 		<child link="R_hip" />
-		<axis xyz="0 0 -1" />
+		<axis xyz="0 0 1" />
 		<limit lower="-0.55" upper="0.55" effort="20.0" velocity="20.0" />
 	</joint>
@@ -257,6 +257,6 @@
 		<parent link="R_hip" />
 		<child link="R_hip2" />
-		<axis xyz="0 0 -1" />
-		<limit lower="-0.18" upper="0.48" effort="20.0" velocity="20.0" />
+		<axis xyz="0 0 1" />
+		<limit lower="-0.48" upper="0.18" effort="20.0" velocity="20.0" />
 	</joint>
 	<link name="R_thigh">
@@ -283,9 +283,9 @@
 	</link>
 	<joint name="R_thigh_joint" type="revolute">
-		<origin xyz="0.0161 0 0.039" rpy="-1.5708 0 1.5708" />
+		<origin xyz="0.0161 0 0.039" rpy="-1.5708 -0.25 1.5708" />
 		<parent link="R_hip2" />
 		<child link="R_thigh" />
-		<axis xyz="0 0 -1" />
-		<limit lower="-0.44" upper="1.0" effort="20.0" velocity="20.0" />
+		<axis xyz="0 0 1" />
+		<limit lower="-1.0" upper="0.44" effort="20.0" velocity="20.0" />
 	</joint>
 	<link name="R_calf">
@@ -312,9 +312,9 @@
 	</link>
 	<joint name="R_calf_joint" type="revolute">
-		<origin xyz="0.15 0 0.0161" rpy="3.1416 0 0" />
+		<origin xyz="0.15 0 0.0161" rpy="3.1416 0 0.5" />
 		<parent link="R_thigh" />
 		<child link="R_calf" />
 		<axis xyz="0 0 1" />
-		<limit lower="-2.0" upper="0" effort="20.0" velocity="20.0" />
+		<limit lower="-1.7" upper="0" effort="20.0" velocity="20.0" />
 	</joint>
 	<link name="R_toe">
@@ -341,5 +341,5 @@
 	</link>
 	<joint name="R_toe_joint" type="revolute">
-		<origin xyz="0.16 0 0" rpy="3.1416 0 1.5708" />
+		<origin xyz="0.16 0 0" rpy="3.1416 0 1.8208" />
 		<parent link="R_calf" />
 		<child link="R_toe" />

Commit message: add 20 dof robot urdf

File: urdf/livelybot_urdf.urdf (robot description, URDF)
Before this commit: robot livelybot_urdf, 12 links, 11 joints
Links:
- removed link L_calf
- removed link L_hip
- removed link L_hip2
- removed link L_thigh
- removed link L_toe
- removed link R_calf
- removed link R_hip
- removed link R_hip2
- removed link R_thigh
- removed link R_toe
- removed link base_link
- removed link imu_link
- added link body, mass 1.65184295519328; collision mesh filename=package://livelybot_urdf/meshes/body.STL; visual mesh filename=package://livelybot_urdf/meshes/body.STL
- added link youshou1, mass 0.0981089714370753; collision mesh filename=package://livelybot_urdf/meshes/youshou1.STL; visual mesh filename=package://livelybot_urdf/meshes/youshou1.STL
- added link youshou2, mass 0.140066448116616; collision mesh filename=package://livelybot_urdf/meshes/youshou2.STL; visual mesh filename=package://livelybot_urdf/meshes/youshou2.STL
- added link youshou3, mass 0.124842254477786; collision mesh filename=package://livelybot_urdf/meshes/youshou3.STL; visual mesh filename=package://livelybot_urdf/meshes/youshou3.STL
- added link youshou4, mass 0.0490685665290975; collision mesh filename=package://livelybot_urdf/meshes/youshou4.STL; visual mesh filename=package://livelybot_urdf/meshes/youshou4.STL
- added link youtui1, mass 0.119463468383066; collision mesh filename=package://livelybot_urdf/meshes/youtui1.STL; visual mesh filename=package://livelybot_urdf/meshes/youtui1.STL
- added link youtui2, mass 0.250906808760741; collision mesh filename=package://livelybot_urdf/meshes/youtui2.STL; visual mesh filename=package://livelybot_urdf/meshes/youtui2.STL
- added link youtui3, mass 0.112705995385217; collision mesh filename=package://livelybot_urdf/meshes/youtui3.STL; visual mesh filename=package://livelybot_urdf/meshes/youtui3.STL
- added link youtui4, mass 0.274677354729083; collision mesh filename=package://livelybot_urdf/meshes/youtui4.STL; visual mesh filename=package://livelybot_urdf/meshes/youtui4.STL
- added link youtui5, mass 0.00886465357060093; collision mesh filename=package://livelybot_urdf/meshes/youtui5.STL; visual mesh filename=package://livelybot_urdf/meshes/youtui5.STL
- added link youtui6, mass 0.180326384410632; collision mesh filename=package://livelybot_urdf/meshes/youtui6.STL; visual mesh filename=package://livelybot_urdf/meshes/youtui6.STL
- added link zuoshou1, mass 0.0936721850648488; collision mesh filename=package://livelybot_urdf/meshes/zuoshou1.STL; visual mesh filename=package://livelybot_urdf/meshes/zuoshou1.STL
- added link zuoshou2, mass 0.140066448116616; collision mesh filename=package://livelybot_urdf/meshes/zuoshou2.STL; visual mesh filename=package://livelybot_urdf/meshes/zuoshou2.STL
- added link zuoshou3, mass 0.124842254477786; collision mesh filename=package://livelybot_urdf/meshes/zuoshou3.STL; visual mesh filename=package://livelybot_urdf/meshes/zuoshou3.STL
- added link zuoshou4, mass 0.0490685665290976; collision mesh filename=package://livelybot_urdf/meshes/zuoshou4.STL; visual mesh filename=package://livelybot_urdf/meshes/zuoshou4.STL
- added link zuotui1, mass 0.119463468383065; collision mesh filename=package://livelybot_urdf/meshes/zuotui1.STL; visual mesh filename=package://livelybot_urdf/meshes/zuotui1.STL
- added link zuotui2, mass 0.250906808479768; collision mesh filename=package://livelybot_urdf/meshes/zuotui2.STL; visual mesh filename=package://livelybot_urdf/meshes/zuotui2.STL
- added link zuotui3, mass 0.109881075271107; collision mesh filename=package://livelybot_urdf/meshes/zuotui3.STL; visual mesh filename=package://livelybot_urdf/meshes/zuotui3.STL
- added link zuotui4, mass 0.274677354729084; collision mesh filename=package://livelybot_urdf/meshes/zuotui4.STL; visual mesh filename=package://livelybot_urdf/meshes/zuotui4.STL
- added link zuotui5, mass 0.00886465357060083; collision mesh filename=package://livelybot_urdf/meshes/zuotui5.STL; visual mesh filename=package://livelybot_urdf/meshes/zuotui5.STL
- added link zuotui6, mass 0.174974482297595; collision mesh filename=package://livelybot_urdf/meshes/zuotui6.STL; visual mesh filename=package://livelybot_urdf/meshes/zuotui6.STL
Joints:
- removed joint L_calf_joint
- removed joint L_hip2_joint
- removed joint L_hip_joint
- removed joint L_thigh_joint
- removed joint L_toe_joint
- removed joint R_calf_joint
- removed joint R_hip2_joint
- removed joint R_hip_joint
- removed joint R_thigh_joint
- removed joint R_toe_joint
- removed joint base_imu_joint
- added joint youshou1: type revolute, parent body, child youshou1, origin xyz=0.0855789473684193 -0.0138454412666174 -0.0364999999999999 rpy=1.5707963267949 0 1.5707963267949, axis 0 0 1, limit lower=0 upper=0 effort=0 velocity=0
- added joint youshou2: type revolute, parent youshou1, child youshou2, origin xyz=0.0315278736990495 0.001927065256896 0.0319210526315811 rpy=0 1.5707963267949 0, axis 0 0 -1, limit lower=0 upper=0 effort=0 velocity=0
- added joint youshou3: type revolute, parent youshou2, child youshou3, origin xyz=0 -0.0709270652568963 -0.0291824324324326 rpy=1.5707963267949 0 0, axis 0 0 1, limit lower=0 upper=0 effort=0 velocity=0
- added joint youshou4: type revolute, parent youshou3, child youshou4, origin xyz=-0.024078947368421 -0.0023454412666174 0.0959999999999999 rpy=-1.5707963267949 0 1.5707963267949, axis 0 0 -1, limit lower=0 upper=0 effort=0 velocity=0
- added joint youtui1: type revolute, parent body, child youtui1, origin xyz=0.0750000405019333 -0.00836285444900997 -0.237429264502804 rpy=-3.14159265358979 0 0, axis 0 0 -1, limit lower=0 upper=0 effort=0 velocity=0
- added joint youtui2: type revolute, parent youtui1, child youtui2, origin xyz=0 0.0387571455509902 0.0525707354971963 rpy=1.5707963267949 0 0, axis 0 0 -1, limit lower=0 upper=0 effort=0 velocity=0
- added joint youtui3: type revolute, parent youtui2, child youtui3, origin xyz=-0.01705 0 0.04 rpy=3.14159265358979 1.5707963267949 0, axis 0 0 -1, limit lower=0 upper=0 effort=0 velocity=0
- added joint youtui4: type revolute, parent youtui3, child youtui4, origin xyz=-0.0113285898146951 -0.149153520094698 -0.0292 rpy=0 0 3.14159265358979, axis 0 0 -1, limit lower=0 upper=0 effort=0 velocity=0
- added joint youtui5: type revolute, parent youtui4, child youtui5, origin xyz=0 0.16 -0.00406906067441093 rpy=3.14159265358979 0 0, axis 0 0 1, limit lower=0 upper=0 effort=0 velocity=0
- added joint youtui6: type revolute, parent youtui5, child youtui6, origin xyz=0.0119556565820659 0 -0.0153997083546931 rpy=3.14159265358979 1.5707963267949 0, axis 0 0 -1, limit lower=0 upper=0 effort=0 velocity=0
- added joint zuoshou1: type revolute, parent body, child zuoshou1, origin xyz=-0.0855789473684207 -0.0138454412666155 -0.0364999999999966 rpy=-1.5707963267949 0 1.5707963267949, axis 0 0 1, limit lower=0 upper=0 effort=0 velocity=0
- added joint zuoshou2: type revolute, parent zuoshou1, child zuoshou2, origin xyz=0.0315278736990499 -0.00192706525689325 0.031921052631579 rpy=0 1.5707963267949 0, axis 0 0 -1, limit lower=0 upper=0 effort=0 velocity=0
- added joint zuoshou3: type revolute, parent zuoshou2, child zuoshou3, origin xyz=0 0.0709270652568965 -0.0291824324324343 rpy=-1.5707963267949 0 0, axis 0 0 1, limit lower=0 upper=0 effort=0 velocity=0
- added joint zuoshou4: type revolute, parent zuoshou3, child zuoshou4, origin xyz=-0.0241522904948619 0.00140130830231822 0.0959999999999999 rpy=1.5707963267949 0 -1.5707963267949, axis 0 0 -1, limit lower=0 upper=0 effort=0 velocity=0
- added joint zuotui1: type revolute, parent body, child zuotui1, origin xyz=-0.0749999594980665 -0.00836285444900986 -0.237429264502804 rpy=3.14159265358979 0 -3.14159265358979, axis 0 0 -1, limit lower=0 upper=0 effort=0 velocity=0
- added joint zuotui2: type revolute, parent zuotui1, child zuotui2, origin xyz=0 -0.0387571455509903 0.052570735497196 rpy=-1.5707963267949 0 0, axis 0 0 -1, limit lower=0 upper=0 effort=0 velocity=0
- added joint zuotui3: type revolute, parent zuotui2, child zuotui3, origin xyz=-0.0170499999999989 0 0.0400000000000003 rpy=3.14159265358979 1.5707963267949 0, axis 0 0 -1, limit lower=0 upper=0 effort=0 velocity=0
- added joint zuotui4: type revolute, parent zuotui3, child zuotui4, origin xyz=-0.0120000000000001 0.149519229532525 -0.0292 rpy=0 0 3.14159265358979, axis 0 0 -1, limit lower=0 upper=0 effort=0 velocity=0
- added joint zuotui5: type revolute, parent zuotui4, child zuotui5, origin xyz=0 -0.159999999999994 -0.00334999999999118 rpy=3.14159265358979 0 0, axis 0 0 1, limit lower=0 upper=0 effort=0 velocity=0
- added joint zuotui6: type revolute, parent zuotui5, child zuotui6, origin xyz=0.0119556565820631 0 -0.0155002916453069 rpy=3.14159265358979 1.5707963267949 0, axis 0 0 -1, limit lower=0 upper=0 effort=0 velocity=0
