Commit message: update model

File: urdf/livelybot_urdf.urdf (robot description, URDF)
Before this commit: robot livelybot_urdf, 21 links, 20 joints
Links:
- removed link body
- removed link youshou1
- removed link youshou2
- removed link youshou3
- removed link youshou4
- removed link youtui1
- removed link youtui2
- removed link youtui3
- removed link youtui4
- removed link youtui5
- removed link youtui6
- removed link zuoshou1
- removed link zuoshou2
- removed link zuoshou3
- removed link zuoshou4
- removed link zuotui1
- removed link zuotui2
- removed link zuotui3
- removed link zuotui4
- removed link zuotui5
- removed link zuotui6
- added link base_link, mass 2.503; collision mesh filename=package://livelybot_urdf/meshes/base_link.STL; visual mesh filename=package://livelybot_urdf/meshes/base_link.STL
- added link l_ankle_pitch_link, mass 0.0088647; collision mesh filename=package://livelybot_urdf/meshes/l_ankle_pitch_link.STL; visual mesh filename=package://livelybot_urdf/meshes/l_ankle_pitch_link.STL
- added link l_ankle_roll_link, mass 0.1749744; collision mesh filename=package://livelybot_urdf/meshes/l_ankle_roll_link.STL; visual mesh filename=package://livelybot_urdf/meshes/l_ankle_roll_link.STL
- added link l_calf_link, mass 0.5043936; collision mesh filename=package://livelybot_urdf/meshes/l_calf_link.STL; visual mesh filename=package://livelybot_urdf/meshes/l_calf_link.STL
- added link l_elbow_link, mass 0.0490686; collision mesh filename=package://livelybot_urdf/meshes/l_elbow_link.STL; visual mesh filename=package://livelybot_urdf/meshes/l_elbow_link.STL
- added link l_hip_roll_link, mass 0.73062; collision mesh filename=package://livelybot_urdf/meshes/l_hip_roll_link.STL; visual mesh filename=package://livelybot_urdf/meshes/l_hip_roll_link.STL
- added link l_hip_yaw_link, mass 0.3593216; collision mesh filename=package://livelybot_urdf/meshes/l_hip_yaw_link.STL; visual mesh filename=package://livelybot_urdf/meshes/l_hip_yaw_link.STL
- added link l_shoulder_pitch_link, mass 0.2085303; collision mesh filename=package://livelybot_urdf/meshes/l_shoulder_pitch_link.STL; visual mesh filename=package://livelybot_urdf/meshes/l_shoulder_pitch_link.STL
- added link l_shoulder_roll_link, mass 0.2549246; collision mesh filename=package://livelybot_urdf/meshes/l_shoulder_roll_link.STL; visual mesh filename=package://livelybot_urdf/meshes/l_shoulder_roll_link.STL
- added link l_shoulder_yaw_link, mass 0.2397004; collision mesh filename=package://livelybot_urdf/meshes/l_shoulder_yaw_link.STL; visual mesh filename=package://livelybot_urdf/meshes/l_shoulder_yaw_link.STL
- added link l_thigh_link, mass 0.1098811; collision mesh filename=package://livelybot_urdf/meshes/l_thigh_link.STL; visual mesh filename=package://livelybot_urdf/meshes/l_thigh_link.STL
- added link r_ankle_pitch_link, mass 0.0088647; collision mesh filename=package://livelybot_urdf/meshes/r_ankle_pitch_link.STL; visual mesh filename=package://livelybot_urdf/meshes/r_ankle_pitch_link.STL
- added link r_ankle_roll_link, mass 0.1803263; collision mesh filename=package://livelybot_urdf/meshes/r_ankle_roll_link.STL; visual mesh filename=package://livelybot_urdf/meshes/r_ankle_roll_link.STL
- added link r_calf_link, mass 0.5043936; collision mesh filename=package://livelybot_urdf/meshes/r_calf_link.STL; visual mesh filename=package://livelybot_urdf/meshes/r_calf_link.STL
- added link r_elbow_link, mass 0.0490686; collision mesh filename=package://livelybot_urdf/meshes/r_elbow_link.STL; visual mesh filename=package://livelybot_urdf/meshes/r_elbow_link.STL
- added link r_hip_roll_link, mass 0.7306; collision mesh filename=package://livelybot_urdf/meshes/r_hip_roll_link.STL; visual mesh filename=package://livelybot_urdf/meshes/r_hip_roll_link.STL
- added link r_hip_yaw_link, mass 0.3593; collision mesh filename=package://livelybot_urdf/meshes/r_hip_yaw_link.STL; visual mesh filename=package://livelybot_urdf/meshes/r_hip_yaw_link.STL
- added link r_shoulder_pitch_link, mass 0.2129671; collision mesh filename=package://livelybot_urdf/meshes/r_shoulder_pitch_link.STL; visual mesh filename=package://livelybot_urdf/meshes/r_shoulder_pitch_link.STL
- added link r_shoulder_roll_link, mass 0.2549246; collision mesh filename=package://livelybot_urdf/meshes/r_shoulder_roll_link.STL; visual mesh filename=package://livelybot_urdf/meshes/r_shoulder_roll_link.STL
- added link r_shoulder_yaw_link, mass 0.2397004; collision mesh filename=package://livelybot_urdf/meshes/r_shoulder_yaw_link.STL; visual mesh filename=package://livelybot_urdf/meshes/r_shoulder_yaw_link.STL
- added link r_thigh_link, mass 0.10988; collision mesh filename=package://livelybot_urdf/meshes/r_thigh_link.STL; visual mesh filename=package://livelybot_urdf/meshes/r_thigh_link.STL
Joints:
- removed joint youshou1
- removed joint youshou2
- removed joint youshou3
- removed joint youshou4
- removed joint youtui1
- removed joint youtui2
- removed joint youtui3
- removed joint youtui4
- removed joint youtui5
- removed joint youtui6
- removed joint zuoshou1
- removed joint zuoshou2
- removed joint zuoshou3
- removed joint zuoshou4
- removed joint zuotui1
- removed joint zuotui2
- removed joint zuotui3
- removed joint zuotui4
- removed joint zuotui5
- removed joint zuotui6
- added joint l_ankle_pitch_joint: type revolute, parent l_calf_link, child l_ankle_pitch_link, origin xyz=0 0 -0.16 rpy=0 0 0, axis 0 1 0, limit lower=-3.14 upper=3.14 effort=21 velocity=21
- added joint l_ankle_roll_joint: type revolute, parent l_ankle_pitch_link, child l_ankle_roll_link, origin xyz=0 0 0 rpy=0 0 0, axis 1 0 0, limit lower=-3.14 upper=3.14 effort=21 velocity=21
- added joint l_calf_link: type revolute, parent l_thigh_link, child l_calf_link, origin xyz=0.012 0 -0.14952 rpy=0 0 0, axis 0 1 0, limit lower=-3.14 upper=3.14 effort=21 velocity=21
- added joint l_elbow_joint: type revolute, parent l_shoulder_yaw_link, child l_elbow_link, origin xyz=0 0.024 -0.091483 rpy=0 0 0, axis 0 1 0, limit lower=-3.14 upper=3.14 effort=21 velocity=21
- added joint l_hip_roll_joint: type revolute, parent l_hip_yaw_link, child l_hip_roll_link, origin xyz=-0.037 0 -0.049 rpy=0 0 0, axis 1 0 0, limit lower=-3.14 upper=3.14 effort=21 velocity=21
- added joint l_hip_yaw_joint: type revolute, parent base_link, child l_hip_yaw_link, origin xyz=0 0.075 0 rpy=0 0 0, axis 0 0 1, limit lower=-3.14 upper=3.14 effort=21 velocity=21
- added joint l_shoulder_pitch_joint: type revolute, parent base_link, child l_shoulder_pitch_link, origin xyz=-0.00237999999999805 0.0854999999999995 0.204500000000003 rpy=1.5707963267949 0 0, axis 0 0 -1, limit lower=-3.14 upper=3.14 effort=21 velocity=21
- added joint l_shoulder_roll_joint: type revolute, parent l_shoulder_pitch_link, child l_shoulder_roll_link, origin xyz=0.024 0 -0.032 rpy=-1.5708 0 0, axis 1 0 0, limit lower=-3.14 upper=3.14 effort=21 velocity=21
- added joint l_shoulder_yaw_joint: type revolute, parent l_shoulder_roll_link, child l_shoulder_yaw_link, origin xyz=-0.024 0 -0.071 rpy=0 0 0, axis 0 0 1, limit lower=-3.14 upper=3.14 effort=21 velocity=21
- added joint l_thigh_joint: type revolute, parent l_hip_roll_link, child l_thigh_link, origin xyz=0.039 0 0 rpy=0 0 0, axis 0 1 0, limit lower=-3.14 upper=3.14 effort=21 velocity=21
- added joint r_ankle_pitch_joint: type revolute, parent r_calf_link, child r_ankle_pitch_link, origin xyz=0 0 -0.16 rpy=0 0 0, axis 0 1 0, limit lower=-3.14 upper=3.14 effort=21 velocity=21
- added joint r_ankle_roll_joint: type revolute, parent r_ankle_pitch_link, child r_ankle_roll_link, origin xyz=0 -0.00081906 0 rpy=0 0 0, axis 1 0 0, limit lower=-3.14 upper=3.14 effort=21 velocity=21
- added joint r_calf_joint: type revolute, parent r_thigh_link, child r_calf_link, origin xyz=0.011329 0 -0.14915 rpy=0 0 0, axis 0 1 0, limit lower=-3.14 upper=3.14 effort=21 velocity=21
- added joint r_elbow_joint: type revolute, parent r_shoulder_yaw_link, child r_elbow_link, origin xyz=0.010624 -0.024 -0.094 rpy=0 0 0, axis 0 1 0, limit lower=-3.14 upper=3.14 effort=21 velocity=21
- added joint r_hip_roll_joint: type revolute, parent r_hip_yaw_link, child r_hip_roll_link, origin xyz=-0.037 0 -0.049 rpy=0 0 0, axis 1 0 0, limit lower=-3.14 upper=3.14 effort=21 velocity=21
- added joint r_hip_yaw_joint: type revolute, parent base_link, child r_hip_yaw_link, origin xyz=0 -0.075 0 rpy=0 0 0, axis 0 0 1, limit lower=-3.14 upper=3.14 effort=21 velocity=21
- added joint r_shoulder_pitch_joint: type revolute, parent base_link, child r_shoulder_pitch_link, origin xyz=-0.00238 -0.0855 0.2045 rpy=0 0 0, axis 0 1 0, limit lower=-3.14 upper=3.14 effort=21 velocity=21
- added joint r_shoulder_roll_joint: type revolute, parent r_shoulder_pitch_link, child r_shoulder_roll_link, origin xyz=0.024 -0.028574 0 rpy=0 0 0, axis 1 0 0, limit lower=-3.14 upper=3.14 effort=21 velocity=21
- added joint r_shoulder_yaw_joint: type revolute, parent r_shoulder_roll_link, child r_shoulder_yaw_link, origin xyz=-0.024 0 -0.071 rpy=0 0 0, axis 0 0 1, limit lower=-3.14 upper=3.14 effort=21 velocity=21
- added joint r_thigh_joint: type revolute, parent r_hip_roll_link, child r_thigh_link, origin xyz=0.039 0 0 rpy=0 0 0, axis 0 1 0, limit lower=-3.14 upper=3.14 effort=21 velocity=21
